File: schematics/DRAM Board.kicad_pcb (KiCad board)
At the start: 2 copper layers, 99.1 x 27.9 mm, 46 parts, among them U1 IS41C16257, U2 IS41C16257

Commit message: Add files via upload
Parts:
- moved C1 53.0 mm to (192.7, 49.8)
- moved C2 53.0 mm to (199.1, 49.8)
- moved U1 53.0 mm to (196.5, 41.5)
- moved C3 53.0 mm to (192.7, 33.3)
- moved C6 48.8 mm to (220.7, 33.3)
- moved C4 48.7 mm to (220.7, 49.8)
- moved C5 48.7 mm to (227.0, 49.8)
- moved U2 48.7 mm to (224.5, 41.5)
- moved vcc_u23 14.0 mm to (168.4, 97.3)
- moved vcc_u17 0.10 mm to (193.6, 97.3)
Routing:
- net /vcc5: track 203.4 -> 254.0 mm
- net /d14: track 62.7 -> 110.9 mm
- net /a2: track 93.1 -> 136.0 mm, vias 1 -> 2
- net /a3: track 91.6 -> 134.2 mm, vias 2 -> 3
- net /d12: track 65.0 -> 104.9 mm
- net /d13: track 71.3 -> 110.4 mm
- net /d15: track 70.2 -> 108.7 mm
- net /a6: track 84.1 -> 121.4 mm
- net /a1: track 86.5 -> 123.3 mm, vias 0 -> 3
- net /a8: track 79.3 -> 115.3 mm
- net /a5: track 86.8 -> 122.1 mm
- net /a4: track 89.3 -> 123.9 mm
- net /_bras0: track 42.7 -> 77.2 mm, vias 1 -> 2
- net /_ucas: track 78.5 -> 112.5 mm, vias 0 -> 3
- net /d9: track 57.3 -> 89.2 mm, vias 2 -> 1
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Other:
- board size 99.1 x 27.9 mm -> 99.1 x 69.8 mm
